Commit message: feat: support hand-side-aware 28-DoF training

File: sim/manorl/runtime_assets/hand/mano_hand.urdf (robot description, URDF)
Before this commit: robot mano_hand, 28 links, 27 joints
Links:
- added link thumb_cmc_flex, mass 0.001
- added link thumb_mcp_flex, mass 0.001
- link index_dip: geometry collision mesh filename=meshes/index3.stl; visual mesh filename=meshes/visual_index3.stl
- link middle_dip: geometry collision mesh filename=meshes/middle3.stl; visual mesh filename=meshes/visual_middle3.stl
- link pinky_dip: geometry collision mesh filename=meshes/pinky3.stl; visual mesh filename=meshes/visual_pinky3.stl
- link ring_dip: geometry collision mesh filename=meshes/ring3.stl; visual mesh filename=meshes/visual_ring3.stl
- link thumb_ip: geometry collision mesh filename=meshes/thumb3.stl; visual mesh filename=meshes/visual_thumb3.stl
Joints:
- removed joint j1_thumb_mcp
- added joint j1_thumb_cmc_twist: type revolute, parent thumb_cmc_flex, child thumb_cmc, origin xyz=0 0 0 rpy=0 0 0, axis 0.11813027 0.24257056 -0.9629147, limit lower=-1.5708 upper=1.5708 effort=100.0 velocity=100.0
- added joint j1_thumb_mcp_abd: type revolute, parent thumb_mcp_flex, child thumb_mcp, origin xyz=0 0 0 rpy=0 0 0, axis -0.5716182768686316 -0.4705844355444832 -0.6721628036220215, limit lower=-0.7 upper=0.7 effort=100.0 velocity=100.0
- added joint j1_thumb_mcp_flex: type revolute, parent thumb_cmc, child thumb_mcp_flex, origin xyz=-0.019956063 0.0012230668 0.024574943 rpy=0 0 0, axis 0.3696764866888757 -0.8790409917024125 0.3010419075414728, limit lower=0.0 upper=1.745 effort=100.0 velocity=100.0
- joint j1_thumb_cmc_flex: child thumb_cmc -> thumb_cmc_flex
- joint j1_thumb_ip: axis 0.3696764866888756 -0.8790409917024126 0.3010419075414728 -> 0.3696764866888757 -0.8790409917024125 0.3010419075414728
- joint j2_index_dip: axis -0.007558282177929704 -0.0004672015231318582 0.9999713266355468 -> -0.007558282177929706 -0.0004672015231318583 0.999971326635547
- joint j2_index_mcp_flex: axis -0.007558282177929704 -0.0004672015231318582 0.9999713266355468 -> -0.007558282177929706 -0.0004672015231318583 0.999971326635547
- joint j2_index_pip: axis -0.007558282177929704 -0.0004672015231318582 0.9999713266355468 -> -0.007558282177929706 -0.0004672015231318583 0.999971326635547
